File: Hardware/PolyMorphFC_V0/PolyMorphFC_V0.kicad_sch (KiCad schematic)
At the start: 1 part, among them U1 STM32F405RGTx

Commit message: FOC Controller Board Schematic OK
Other:
- sheet Positionig Region renamed Positioning Region
- sheet Positioning Region ports: added BARO_INT, IMU_CS, IMU_INT, IMU_MISO, IMU_MOSI, IMU_SCK, MAG_DT_RDY, MAG_RST, POS_SCL, POS_SDA; removed none
Changed lines of the file:
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@@
 	)
 	(sheet
-		(at 32.512 149.606)
-		(size 71.628 37.084)
+		(at 20.32 21.082)
+		(size 33.528 37.084)
 		(exclude_from_sim no)
 		(in_bom yes)
@@
 			(color 0 0 0 0.0000)
 		)
-		(property "Sheetname" "Positionig Region"
-			(at 32.512 148.8944 0)
+		(property "Sheetname" "Positioning Region"
+			(at 20.32 20.3704 0)
 			(effects
 				(font
@@
 		)
 		(property "Sheetfile" "positioning_region.kicad_sch"
-			(at 32.512 187.2746 0)
+			(at 20.32 58.7506 0)
 			(effects
 				(font
@@
 			)
 		)
+		(pin "BARO_INT" input
+			(at 53.848 45.466 0)
+			(effects
+				(font
+					(size 1.27 1.27)
+				)
+				(justify right)
+			)
+		)
+		(pin "IMU_CS" input
+			(at 53.848 39.116 0)
+			(effects
+				(font
+					(size 1.27 1.27)
+				)
+				(justify right)
+			)
+		)
+		(pin "IMU_INT" input
+			(at 53.848 50.546 0)
+			(effects
+				(font
+					(size 1.27 1.27)
+				)
+				(justify right)
+			)
+		)
+		(pin "IMU_MISO" input
+			(at 53.848 34.036 0)
+			(effects
+				(font
+					(size 1.27 1.27)
+				)
+				(justify right)
+			)
+		)
+		(pin "IMU_MOSI" input
+			(at 53.848 31.496 0)
+			(effects
+				(font
+					(size 1.27 1.27)
+				)
+				(justify right)
+			)
+		)
+		(pin "IMU_SCK" input
+			(at 53.848 36.576 0)
+			(effects
+				(font
+					(size 1.27 1.27)
+				)
+				(justify right)
+			)
+		)
+		(pin "MAG_DT_RDY" input
+			(at 53.848 48.006 0)
+			(effects
+				(font
+					(size 1.27 1.27)
+				)
+				(justify right)
+			)
+		)
+		(pin "MAG_RST" input
+			(at 53.848 55.626 0)
+			(effects
+				(font
+					(size 1.27 1.27)
+				)
+				(justify right)
+			)
+		)
+		(pin "POS_SCL" input
+			(at 53.848 25.146 0)
+			(effects
+				(font
+					(size 1.27 1.27)
+				)
+				(justify right)
+			)
+		)
+		(pin "POS_SDA" input
+			(at 53.848 22.606 0)
+			(effects
+				(font
+					(size 1.27 1.27)
+				)
+				(justify right)
+			)
+		)
