File: Hardware/PolyMorphFC_V0/positioning_region.kicad_sch (KiCad schematic)
At the start: 12 parts, among them U3 ICM42688-P

Commit message: FOC Controller Board Schematic OK
Parts:
- removed C3: 0.1uF, symbol Device:C_Small
- removed R1, R2: 10kΩ, symbol Device:R
- removed R3, R4: 4.7kΩ, symbol Device:R
- added C10, C11: 0.1uF, symbol Device:C
- added C9: 4.7uF, symbol Device:C
- added R6, R7: 4.7kΩ, symbol Device:R
- added U3: IST8310, Package_LGA:LGA-16_3x3mm_P0.5mm, symbol Sensor_Magnetic:IST8310
- U2: renamed from 1; footprint Adafruit BMP388:BMP388 -> Package_LGA:ST_HLGA-10_2x2mm_P0.5mm_LayoutBorder3x2y
Connections:
- net +3V3: now also C4.2, U2.6 (CSB), U3.5 (VDDIO), C10.1, C11.1, R6.1, R7.1, U3.13 (DVDD), U3.2 (AVDD), U3.7 (VPP); no longer C1.1, C1.2, C2.1, C4.1, C5.2, C6.2, U2.3 (GND), U2.8 (GND), U2.9 (GND), U3.10 (RESV), U3.11 (RESV), U3.2 (RESV), U3.3 (RESV), U3.6 (GND), U3.7 (RESV)
- net POS_SCL: now reaches U2.2 (SCK)
- net POS_SCL: now also R7.2, U3.1 (SCL)
- net POS_SDA: now reaches U2.4 (SDI)
- net POS_SDA: now also R6.2, U3.16 (SDA)
- net GND: now reaches U2.5 (SDO)
- net GND: now also C1.2, C2.1, C4.1, C5.2, C6.2, U3.10 (RESV), U3.11 (RESV), U3.2 (RESV), U3.3 (RESV), U3.6 (GND), U3.7 (RESV), C10.2, C11.2, C9.2, U3.11 (VSS), U3.5 (CAD0), U3.6 (CAD1), U3.9 (VSS)
- net IMU_INT: now reaches U3.4 (INT1)
- new net: C9.1, U3.10 (C1)
- new net: C1.1, U2.3 (GND), U2.8 (GND), U2.9 (GND)
- new net MAG_DT_RDY: U3.15 (DRDY)
- new net MAG_RST: U3.14 (~{RST})
